File: dilemma-cirque/dilemma-cirque.kicad_sch (KiCad schematic)
At the start: 9 parts, among them J1 CirqueDB

Commit message: clean up footprints
Parts:
- H1, H2, H3, H4: footprint MountingHole:MountingHole_3.2mm_M3_DIN965_Pad -> footprints:MountingHole_3mm_Pad_thin
Changed lines of the file:
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@@
     (property "Reference" "H3" (id 0) (at 66.294 40.2422 90))
     (property "Value" "MountingHole_Pad" (id 1) (at 66.294 42.7791 90))
-    (property "Footprint" "MountingHole:MountingHole_3.2mm_M3_DIN965_Pad" (id 2) (at 67.564 45.72 0)
+    (property "Footprint" "footprints:MountingHole_3mm_Pad_thin" (id 2) (at 67.564 45.72 0)
       (effects (font (size 1.27 1.27)) hide)
     )
@@
     (property "Reference" "H1" (id 0) (at 66.294 19.9222 90))
     (property "Value" "MountingHole_Pad" (id 1) (at 66.294 22.4591 90))
-    (property "Footprint" "MountingHole:MountingHole_3.2mm_M3_DIN965_Pad" (id 2) (at 67.564 25.4 0)
+    (property "Footprint" "footprints:MountingHole_3mm_Pad_thin" (id 2) (at 67.564 25.4 0)
       (effects (font (size 1.27 1.27)) hide)
     )
@@
     (property "Reference" "H4" (id 0) (at 66.294 50.4022 90))
     (property "Value" "MountingHole_Pad" (id 1) (at 66.294 52.9391 90))
-    (property "Footprint" "MountingHole:MountingHole_3.2mm_M3_DIN965_Pad" (id 2) (at 67.564 55.88 0)
+    (property "Footprint" "footprints:MountingHole_3mm_Pad_thin" (id 2) (at 67.564 55.88 0)
       (effects (font (size 1.27 1.27)) hide)
     )
@@
     (property "Reference" "H2" (id 0) (at 66.294 30.0822 90))
     (property "Value" "MountingHole_Pad" (id 1) (at 66.294 32.6191 90))
-    (property "Footprint" "MountingHole:MountingHole_3.2mm_M3_DIN965_Pad" (id 2) (at 67.564 35.56 0)
+    (property "Footprint" "footprints:MountingHole_3mm_Pad_thin" (id 2) (at 67.564 35.56 0)
       (effects (font (size 1.27 1.27)) hide)
     )
@@
     )
     (path "/17c88554-b84a-4558-a973-bb4ec16ea7b6"
-      (reference "H1") (unit 1) (value "MountingHole_Pad") (footprint "MountingHole:MountingHole_3.2mm_M3_DIN965_Pad")
+      (reference "H1") (unit 1) (value "MountingHole_Pad") (footprint "footprints:MountingHole_3mm_Pad_thin")
     )
     (path "/f515a122-b419-4a67-b625-1d6b443c7959"
-      (reference "H2") (unit 1) (value "MountingHole_Pad") (footprint "MountingHole:MountingHole_3.2mm_M3_DIN965_Pad")
+      (reference "H2") (unit 1) (value "MountingHole_Pad") (footprint "footprints:MountingHole_3mm_Pad_thin")
     )
     (path "/0cee515e-bff0-441c-808f-5c7f575531ab"
-      (reference "H3") (unit 1) (value "MountingHole_Pad") (footprint "MountingHole:MountingHole_3.2mm_M3_DIN965_Pad")
+      (reference "H3") (unit 1) (value "MountingHole_Pad") (footprint "footprints:MountingHole_3mm_Pad_thin")
     )
     (path "/632c8793-0a5e-4b9e-8fad-8505a760b4eb"
-      (reference "H4") (unit 1) (value "MountingHole_Pad") (footprint "MountingHole:MountingHole_3.2mm_M3_DIN965_Pad")
+      (reference "H4") (unit 1) (value "MountingHole_Pad") (footprint "footprints:MountingHole_3mm_Pad_thin")
     )
     (path "/0c15bea0-7570-445f-946c-68b28e4351f3"
